File: midi controller.sch (KiCad schematic (older format))
At the start: 45 parts, among them J1 Conn_01x04, SW1 SW_Push, SW2 SW_Push, SW3 SW_Push, SW4 SW_Push, U1 Teensy4.0-d

Commit message: updated the fader and switch devices
Parts:
- removed SVR1, SVR2, SVR3, SVR4: RS6011SP6003, SamacSys_Parts:RS6011SP6003, symbol RS6011SP6003:RS6011SP6003
- added SVR1, SVR2, SVR3, SVR4: PTA6043-2015CPB103, PTA6043-2015CPB103:PTA60432015CPB103, symbol PTA6043-2015CPB103:PTA6043-2015CPB103
- SW1, SW2, SW3, SW4: footprint midi controller:1543-650-149 -> midi controller:800SP9B7M2QE
- TB1, TB2: symbol midi-components:CD74HC4067 -> midi-controller-rescue:CD74HC4067-midi-components
- U1: symbol teensy:Teensy4.0-d -> midi-controller-rescue:Teensy4.0-d-teensy
- VR1, VR10, VR11, VR12, VR13, VR14, VR15, VR16, VR17, VR18, VR19, VR2, VR20, VR3, VR4, VR5, VR6, VR7, VR8, VR9: symbol PTV09A-4025F-B103:PTV09A-4025F-B103 -> midi-controller-rescue:PTV09A-4025F-B103-PTV09A-4025F-B103
Connections:
- net 3V3: now also SVR1.3 (CW), SVR2.3 (CW), SVR3.3 (CW), SVR4.3 (CW)
- net GND: now also SVR1.1 (CCW), SVR2.1 (CCW), SVR3.1 (CCW), SVR4.1 (CCW)
- net SL1: now also SVR1.2 (WIPER)
- net SL2: now also SVR2.2 (WIPER)
- net SL3: now also SVR3.2 (WIPER)
- net SL4: now also SVR4.2 (WIPER)
- no-connect marks 89 -> 85
